Commit message: add camera and finalize values

File: description/gantry_description.urdf (robot description, URDF)
Before this commit: robot gantry_bot, 1 links, 0 joints
Links:
- added link front_cam_link
- link base_link: geometry visual cylinder length=${pillar_length} radius=${pillar_diameter/2}
Joints:
- added joint front_cam_identity: type fixed, parent camera_link, child front_cam_link

Commit message: add second camera

File: description/gantry_description.urdf (robot description, URDF)
Before this commit: robot gantry_bot, 1 links, 0 joints
Links:
- link base_link: geometry visual cylinder length=${pillar_length} radius=${pillar_diameter/2}

Commit message: tune values

File: description/gantry_description.urdf (robot description, URDF)
Before this commit: robot gantry_bot, 2 links, 1 joints
Links:
- removed link front_cam_link
Joints:
- removed joint front_cam_identity
